Commit message: adjusting for use of gripper

File: robot_description/maci.urdf (robot description, URDF)
Before this commit: robot maci, 13 links, 12 joints
Links:
- added link left_inner_finger, mass 0.0104003125914103; collision mesh filename=file:///workspace/install/robotiq_2f_140_gripper_visualizat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; visual mesh filename=file:///workspace/install/robotiq_2f_140_gripper_visualizat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
- added link left_inner_finger_pad; collision box size=0.03 0.07 0.0075; visual box size=0.027 0.065 0.0075
- added link left_inner_knuckle, mass 0.0271177346495152; collision mesh filename=file:///workspace/install/robotiq_2f_140_gripper_visualizat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; visual mesh filename=file:///workspace/install/robotiq_2f_140_gripper_visualizat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
- added link left_outer_finger, mass 0.022614240507152; collision mesh filename=file:///workspace/install/robotiq_2f_140_gripper_visualizat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; visual mesh filename=file:///workspace/install/robotiq_2f_140_gripper_visualizat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
- added link left_outer_knuckle, mass 0.00853198276973456; collision mesh filename=file:///workspace/install/robotiq_2f_140_gripper_visualizat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; visual mesh filename=file:///workspace/install/robotiq_2f_140_gripper_visualizat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
- added link right_inner_finger, mass 0.0104003125914103; collision mesh filename=file:///workspace/install/robotiq_2f_140_gripper_visualizat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; visual mesh filename=file:///workspace/install/robotiq_2f_140_gripper_visualizat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
- added link right_inner_finger_pad; collision box size=0.03 0.07 0.0075; visual box size=0.027 0.065 0.0075
- added link right_inner_knuckle, mass 0.0271177346495152; collision mesh filename=file:///workspace/install/robotiq_2f_140_gripper_visualizat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; visual mesh filename=file:///workspace/install/robotiq_2f_140_gripper_visualizat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
- added link right_outer_finger, mass 0.022614240507152; collision mesh filename=file:///workspace/install/robotiq_2f_140_gripper_visualizat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; visual mesh filename=file:///workspace/install/robotiq_2f_140_gripper_visualizat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
- added link right_outer_knuckle, mass 0.00853198276973456; collision mesh filename=file:///workspace/install/robotiq_2f_140_gripper_visualizat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; visual mesh filename=file:///workspace/install/robotiq_2f_140_gripper_visualizat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
- added link robotiq_arg2f_base_link, mass 0.22652; collision mesh filename=file:///workspace/install/robotiq_2f_140_gripper_visualizat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; visual mesh filename=file:///workspace/install/robotiq_2f_140_gripper_visualizat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
- link ur5_base_link_inertia: geometry collision mesh filename=file:///opt/ros/humble/share/ur_description/meshes/ur5e/col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; visual mesh filename=file:///opt/ros/humble/share/ur_description/meshes/ur5e/vis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
- link ur5_forearm_link: geometry collision mesh filename=file:///opt/ros/humble/share/ur_description/meshes/ur5e/col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; visual mesh filename=file:///opt/ros/humble/share/ur_description/meshes/ur5e/vis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
- link ur5_shoulder_link: geometry collision mesh filename=file:///opt/ros/humble/share/ur_description/meshes/ur5e/col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; visual mesh filename=file:///opt/ros/humble/share/ur_description/meshes/ur5e/vis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
- link ur5_upper_arm_link: geometry collision mesh filename=file:///opt/ros/humble/share/ur_description/meshes/ur5e/col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; visual mesh filename=file:///opt/ros/humble/share/ur_description/meshes/ur5e/vis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
- link ur5_wrist_1_link: geometry collision mesh filename=file:///opt/ros/humble/share/ur_description/meshes/ur5e/col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; visual mesh filename=file:///opt/ros/humble/share/ur_description/meshes/ur5e/vis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
- link ur5_wrist_2_link: geometry collision mesh filename=file:///opt/ros/humble/share/ur_description/meshes/ur5e/col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; visual mesh filename=file:///opt/ros/humble/share/ur_description/meshes/ur5e/vis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
- link ur5_wrist_3_link: geometry collision mesh filename=file:///opt/ros/humble/share/ur_description/meshes/ur5e/col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; visual mesh filename=file:///opt/ros/humble/share/ur_description/meshes/ur5e/vis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
Joints:
- added joint finger_joint: type revolute, parent robotiq_arg2f_base_link, child left_outer_knuckle, origin xyz=0 -0.030601 0.054905 rpy=2.2957963267948966 0 0, axis -1 0 0, limit lower=0 upper=0.7 effort=1000 velocity=2.0
- added joint gripper_connect: type fixed, parent ur5_tool0, child robotiq_arg2f_base_link
- added joint left_inner_finger_joint: type revolute, parent left_outer_finger, child left_inner_finger, origin xyz=0 0.0817554015893473 -0.0282203446692936 rpy=-0.725 0 0, axis 1 0 0, limit lower=0 upper=0.8757 effort=1000 velocity=2.0, mimic joint=finger_joint multiplier=1 offset=0
- added joint left_inner_finger_pad_joint: type fixed, parent left_inner_finger, child left_inner_finger_pad, origin xyz=0 0.0457554015893473 -0.0272203446692936 rpy=0 0 0, axis 0 0 1
- added joint left_inner_knuckle_joint: type revolute, parent robotiq_arg2f_base_link, child left_inner_knuckle, origin xyz=0 -0.0127 0.06142 rpy=2.2957963267948966 0 0.0, axis 1 0 0, limit lower=0 upper=0.8757 effort=1000 velocity=2.0, mimic joint=finger_joint multiplier=-1 offset=0
- added joint left_outer_finger_joint: type fixed, parent left_outer_knuckle, child left_outer_finger, origin xyz=0 0.01821998610742 0.0260018192872234 rpy=0 0 0, axis 1 0 0
- added joint right_inner_finger_joint: type revolute, parent right_outer_finger, child right_inner_finger, origin xyz=0 0.0817554015893473 -0.0282203446692936 rpy=-0.725 0 0, axis 1 0 0, limit lower=0 upper=0.8757 effort=1000 velocity=2.0, mimic joint=finger_joint multiplier=1 offset=0
- added joint right_inner_finger_pad_joint: type fixed, parent right_inner_finger, child right_inner_finger_pad, origin xyz=0 0.0457554015893473 -0.0272203446692936 rpy=0 0 0, axis 0 0 1
- added joint right_inner_knuckle_joint: type revolute, parent robotiq_arg2f_base_link, child right_inner_knuckle, origin xyz=0 0.0127 0.06142 rpy=2.2957963267948966 0 -3.141592653589793, axis 1 0 0, limit lower=0 upper=0.8757 effort=1000 velocity=2.0, mimic joint=finger_joint multiplier=-1 offset=0
- added joint right_outer_finger_joint: type fixed, parent right_outer_knuckle, child right_outer_finger, origin xyz=0 0.01821998610742 0.0260018192872234 rpy=0 0 0, axis 1 0 0
- added joint right_outer_knuckle_joint: type revolute, parent robotiq_arg2f_base_link, child right_outer_knuckle, origin xyz=0 0.030601 0.054905 rpy=2.2957963267948966 0 3.141592653589793, axis 1 0 0, limit lower=0 upper=0.725 effort=1000 velocity=2.0, mimic joint=finger_joint multiplier=-1 offset=0

File: robot_description/maci.urdf.xacro (robot description, xacro)
@@ -8,11 +8,24 @@
     </xacro:ur_robot>
     <link name="world" />
+    <xacro:include filename="$(find robotiq_2f_140_gripper_visualization)/urdf/robotiq_arg2f_140_model.xacro" />
+    <joint name="gripper_connect" type="fixed" >
+        <parent link="ur5_tool0" />
+        <child link="robotiq_arg2f_base_link" />
+    </joint>
+    <ros2_control name="ur5_" type="system">
+        <hardware>
+            <plugin>ign_ros2_control/IgnitionSystem</plugin>
+        </hardware>
+        <joint name="finger_joint">
+            <command_interface name="position"/>
+            <state_interface name="position">
+                <param name="initial_value">0.0</param>
+            </state_interface>
+            <state_interface name="velocity"/>
+        </joint>
+    </ros2_control>
     <gazebo>
         <plugin filename="ign_ros2_control-system" name="ign_ros2_control::IgnitionROS2ControlPlugin">
-            <controller_manager_prefix_node_name>maci</controller_manager_prefix_node_name>
             <parameters>$(find maci)/config/ros2_control.yaml</parameters>
-            <ros>
-                <namespace>maci</namespace>
-            </ros>
         </plugin>
     </gazebo>

Commit message: Adjusting urdf so that gripper works

File: robot_description/maci.urdf (robot description, URDF)
Before this commit: robot maci, 24 links, 23 joints
Joints:
- joint left_inner_finger_joint: mimic joint=finger_joint multiplier=1 offset=0 -> (none)
- joint left_inner_knuckle_joint: limit lower=0 upper=0.8757 effort=1000 velocity=2.0 -> lower=-0.8757 upper=0.8757 effort=1000 velocity=2.0; mimic joint=finger_joint multiplier=-1 offset=0 -> (none)
- joint right_inner_finger_joint: mimic joint=finger_joint multiplier=1 offset=0 -> (none)
- joint right_inner_knuckle_joint: limit lower=0 upper=0.8757 effort=1000 velocity=2.0 -> lower=-0.8757 upper=0.8757 effort=1000 velocity=2.0; mimic joint=finger_joint multiplier=-1 offset=0 -> (none)
- joint right_outer_knuckle_joint: limit lower=0 upper=0.725 effort=1000 velocity=2.0 -> lower=0 upper=-0.725 effort=1000 velocity=2.0; mimic joint=finger_joint multiplier=-1 offset=0 -> (none)
