Commit message: Adjusted controllers for not having inner knuckes

File: robot_description/maci.urdf.xacro (robot description, xacro)
@@ -9,13 +9,10 @@
     <link name="world" />
     <xacro:include filename="$(find robotiq_2f_140_gripper_visualization)/urdf/robotiq_arg2f_140_model.xacro" />
-    <joint name="gripper_connect" type="fixed" >
+    <joint name="gripper_connect" type="fixed">
         <parent link="ur5_tool0" />
         <child link="robotiq_arg2f_base_link" />
     </joint>
-    <ros2_control name="ur5_" type="system">
-        <hardware>
-            <plugin>ign_ros2_control/IgnitionSystem</plugin>
-        </hardware>
-        <joint name="finger_joint">
+    <xacro:macro name="ros2_position_controller" params="joint_name">
+        <joint name="${joint_name}">
             <command_interface name="position"/>
             <state_interface name="position">
@@ -24,4 +21,13 @@
             <state_interface name="velocity"/>
         </joint>
+    </xacro:macro>
+    <ros2_control name="ur5_" type="system">
+        <hardware>
+            <plugin>ign_ros2_control/IgnitionSystem</plugin>
+        </hardware>
+        <xacro:ros2_position_controller joint_name="finger_joint" />
+        <xacro:ros2_position_controller joint_name="left_inner_finger_joint" />
+        <xacro:ros2_position_controller joint_name="right_outer_knuckle_joint" />
+        <xacro:ros2_position_controller joint_name="right_inner_finger_joint" />
     </ros2_control>
     <gazebo>
